Commit message: feat: dynamic posture reference + sim2real fixes (dt, ref posture, hip_roll limits)

File: assets/q1/urdf/q1.urdf (robot description, URDF)
Before this commit: robot YSXSZ, 12 links, 11 joints
Joints:
- joint hip_roll_l: limit lower=-0.3 upper=0.6 effort=60 velocity=10 -> lower=0 upper=0.6 effort=60 velocity=10
- joint hip_roll_r: limit lower=-0.6 upper=0.3 effort=60 velocity=10 -> lower=-0.6 upper=0.0 effort=60 velocity=10
